File: pcb/ch55xRebootTool/ch55xRebootTool.brd (EAGLE design)
At the start: 40.6 x 12 mm, 21 parts, among them IC1 CH443K, IC2 CH443K, U2 CH552G

Commit message: update board
Parts:
- removed X2: (no value), con-yamaichi:USB-A003
- added C3: 0.1uF, rcl:C0805K
- added C4: DNP, rcl:C0805K
- added F2, F3: (no value), adafruit:R1206
- added IC3: 74AHCT1G08DCK, 74xx-little-us:SC70-5
- added JP1: (no value), pinhead:1X03
- added R4: 20K, rcl:R0805
- added R5: 10K, rcl:R0805
- added T3: (no value), zetex:SOT-23
- added USB3, USB5: 292303-1, USB connector:292303-1
- added USB4: ZX62-B-5PA, microusbConnector:MICRO-USB5+6P-SMD-0.65-AB
- moved T2 52.9 mm to (33.7, 15.3), turned to 180 degrees
- moved T1 45.5 mm to (30.1, 15.3), turned to 180 degrees
- moved IC2 26.0 mm to (11.4, 13.8), turned to 270 degrees
- moved IC1 22.8 mm to (11.4, 16.4), turned to 270 degrees
- moved USB2 3.68 mm to (1.52, 20.3)
Connections:
- removed net V_USB_MCU: T1.1
- new net N$4: IC3.4, R4.1
- new net N$5: F3.1, T1.1
- new net N$7: R5.1, T3.1
- new net PERI_D+: IC2.1, USB3.3
- new net PERI_D-: IC1.1, USB3.2
- new net SHIELD: USB3.SH1, USB3.SH2, USB5.SH1, USB5.SH2
- new net TAR_COMP_D+: IC2.3, USB2.3
- new net TAR_COMP_D-: IC1.3, USB2.2
- new net TAR_D+: IC2.4, IC3.2, R5.2, USB4.3, USB5.3
- new net TAR_D-: IC1.4, IC3.1, USB4.2, USB5.2
- new net VBUS_COMP: F2.1, USB2.1
- new net VBUS_TAR: F3.2, USB4.1, USB5.1
- net +5V: now also C3.1, F2.2, IC3.5, T3.2
- net GND: now also C3.2, C4.2, IC3.3, JP1.3, USB2.5, USB3.4, USB4.5, USB5.4
- net P1.1: now also T2.3
- net P1.4: now also T3.3
- net P3.0: now also JP1.1
- net P3.1: now also JP1.2
- net P3.2: now also C4.1, R4.2; no longer T2.3
- net P3.3: now also IC1.6, IC2.6
- net V_USB_PERI: now also USB3.1
Routing:
- net GND: track 61.4 -> 180.1 mm, vias 4 -> 15
- net +5V: track 57.9 -> 116.7 mm, vias 3 -> 10
- net P1.4: track 2.89 -> 54.2 mm, vias 0 -> 3
- net TAR_D+: track 0.00 -> 43.2 mm, vias 0 -> 6
- net TAR_D-: track 0.00 -> 34.9 mm, vias 0 -> 2
- net SHIELD: track 0.00 -> 30.6 mm, vias 0 -> 2
- net PERI_D+: track 0.00 -> 29.2 mm, vias 0 -> 2
- net PERI_D-: track 0.00 -> 28.4 mm, vias 0 -> 2
- net P3.1: track 17.0 -> 45.1 mm, vias 3 -> 4
- net P3.0: track 17.5 -> 45.4 mm
- net P3.2: track 21.5 -> 48.2 mm, vias 3 -> 5
- net VBUS_TAR: track 0.00 -> 24.2 mm
- net P3.3: track 21.2 -> 40.5 mm, vias 1 -> 3
- net P1.1: track 17.2 -> 30.6 mm
- net VBUS_COMP: track 0.00 -> 12.4 mm, vias 0 -> 2
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Other:
- board size 40.6 x 12 mm -> 40.6 x 33 mm
- board text added: "Bootloader Tool"
- board text added: "Deqing Sun, 2021 Try Ch55xduino with this board"
- board text added: "Deqing, 2021"
- board text added: "Helper USB"
- board text added: "P3.3 controls USB switch P3.4 switch power of target P1.1 switch power of peripheral P1.4 controls D+ pullup of target P3.2 senses USB reset"
- board text added: "Peri USB"
- board text added: "RX"
- board text added: "TX"
- board text added: "Target USB"
- board text added: "Target Upload"
- board text removed: "CH552 STICK"
- board text removed: "Deqing Sun, 2020 Try Ch55xduino with this board"
- board text removed: "Deqing, 2020"
